File: Hardware/pmodia-mux/Redesign-8Ch-Mux-Breakout-PMODIA.sch (EAGLE design)
At the start: 30 parts, among them U1 74HC4051BQ, U2 74HC4051BQ, U3 AD5933, U4 AD8606, U5 ADP150, U6 AD8606

Commit message: Add files via upload
Parts:
- removed R10: 300, SparkFun-Resistors:0.3OHM-0805-1/8W-1%
- added X1, X2: BU-SMA-G, con-coax:BU-SMA-G
- C7: value 47nF -> (none)
Connections:
- new net N$10: U4.INA_N, U4.OUTA
- new net N$13: X2.1
- new net N$3: R8.2, R9.2, U6.INA_N
- net GND: now also X1.1, X1.2, X2.2
- net Y0: no longer R10.1
- net Y20: no longer R10.2
- net Z: no longer U4.INA_N, U4.OUTA
- net Z2: no longer R8.2, R9.2, U6.INA_N
Other:
- note added: "CHECK SMA CONNECTOR"

Commit message: Add files via upload
Parts:
- removed C10, C11, C7, C8, C9: (no value), rcl:C-US025-024X044
- removed C5, C6: 0.1uF, rcl:C-US025-024X044
- removed R2, R3, R6, R7: 49.9K, rcl:R-US_0204/7
- removed R4: 20K, rcl:R-US_0204/7
- removed R5: (no value), rcl:R-US_0204/7
- removed R8: 20, rcl:R-US_0204/7
- removed R9: 100K, rcl:R-US_0204/7
- removed X1, X2: BU-SMA-G, con-coax:BU-SMA-G
- added C15, C16, C20, C22, C25: 10uF, rcl:C-USC0805K
- added C17, C18, C21, C23, C24: 0.1uF, rcl:C-USC0805K
- added C19: 47nF, rcl:C-USC0805K
- added R10: 300, SparkFun-Resistors:0.3OHM-0805-1/8W-1%
- added R11, R12, R13, R14: 49.9K, rcl:R-US_R0603
- added R15: 20, rcl:R-US_R0603
- added R16, R18: 20K, rcl:R-US_R0603
- added R17: 100K, rcl:R-US_R0603
- C2, C4: value 10uF -> 0.1uF; device rcl:C-US025-024X044 -> rcl:C-USC0805K
- C3: value 0.1uF -> 10uF; device rcl:C-US025-024X044 -> rcl:C-USC0805K
Connections:
- removed net N$10: U4.INA_N, U4.OUTA
- removed net N$13: X2.1
- removed net N$2: C7.2, R2.1, R3.2, U4.INA_P
- removed net N$7: U3.DGND
- net GND: now also C15.2, C16.2, C17.2, C18.2, C20.2, C21.2, C22.2, C23.1, C24.2, C25.2, R11.2, R14.1, U3.DGND, U4.V_N, U6.V_N; no longer C10.2, C11.2, C5.2, C6.2, C8.2, C9.2, R2.2, R7.1, X1.1, X1.2, X2.2
- net N$1: now also C19.1; no longer C7.1
- net N$11: now also R16.1; no longer R5.2
- net N$3: now also C19.2, R11.1, R12.2, U4.INA_P; no longer R8.2, R9.2, U6.INA_N
- net N$4: now also R13.1, R14.2; no longer R6.1, R7.2
- net N$5: now also R18.2; no longer R4.2
- net N$6: now also R15.2; no longer R8.1
- net N$9: now also R17.2; no longer R9.1
- net VCC: now also C18.1, C23.2, C25.1, C4.1; no longer C2.1, C6.1, C8.1, C9.1
- net VCC3V0: now also C15.1, C16.1, C17.1, C2.1, C20.1, C21.1, C22.1, C24.1, R12.1, R13.2, U4.V_P, U6.V_P; no longer C10.1, C11.1, C4.1, C5.1, R3.1, R6.2
- net VIN: now also R16.2, R18.1; no longer R4.1, R5.1
- net Y0: now also R10.1
- net Y20: now also R10.2
- net Z: now also U4.INA_N, U4.OUTA
- net Z2: now also R15.1, R17.1, U6.INA_N
Other:
- note removed: "CHECK SMA CONNECTOR"
- note removed: "MAKE PMODIA AND BOARD CONNECTIONS PLEASE"
- note removed: "opamp power is separate on the PMODIA schematic, is that good practice????? how to do with the one we have in our schematic (will overlap wires and be a mess)"
- moved on the sheet: C2, C3, C4, U4, U5, U6
