File: Hardware/pmodia-mux/Redesign-8Ch-Mux-Breakout-PMODIA.sch (EAGLE design)
At the start: 31 parts, among them U1 74HC4051BQ, U2 74HC4051BQ, U3 AD5933, U4 AD8606, U5 ADP150

Commit message: Add files via upload
Parts:
- removed JP1: (no value), pinhead:PINHD-2X8
- added X1: FH12-16S-0.5SH, con-hirose:FH12-16S-0.5SH
Connections:
- net Y0: now also X1-8.1; no longer JP1.1
- net Y1: now also X1-7.1; no longer JP1.3
- net Y2: now also X1-6.1; no longer JP1.5
- net Y20: now also X1-9.1; no longer JP1.2
- net Y21: now also X1-10.1; no longer JP1.4
- net Y22: now also X1-11.1; no longer JP1.6
- net Y23: now also X1-12.1; no longer JP1.8
- net Y24: now also X1-13.1; no longer JP1.10
- net Y25: now also X1-14.1; no longer JP1.12
- net Y26: now also X1-15.1; no longer JP1.14
- net Y27: now also X1-16.1; no longer JP1.16
- net Y3: now also X1-5.1; no longer JP1.7
- net Y4: now also X1-4.1; no longer JP1.9
- net Y5: now also X1-3.1; no longer JP1.11
- net Y6: now also X1-2.1; no longer JP1.13
- net Y7: now also X1-1.1; no longer JP1.15
Other:
- note removed: "clean up this crossover"
