File: Hardware/Arduino+SD+DAC/main.brd (EAGLE design)
At the start: 64 x 45.7 mm, 28 parts, among them IC3 4050D, IC4 LP298XS, J1 POWER_JACK, U1 5V, U2 328P, U4 MCP4725, X2 MICROSD

Commit message: Schematic
Parts:
- removed JP6: (no value), pinhead:1X04
- added JP1: (no value), pinhead:1X10
- moved JP4 3.56 mm to (9.14, -4.06)
- moved JP5 3.56 mm to (9.14, -9.65)
Connections:
- removed net N$21: U2.24
- removed net N$24: JP3.5
- new net N$14: JP1.6, U2.12
- new net N$15: JP1.7, U2.13
- new net N$16: JP1.8, U2.14
- new net N$18: JP1.10, U2.16
- new net N$6: JP1.3, U2.4
- new net N$8: JP1.4, U2.5
- new net N$9: JP1.5, U2.11
- new net SS: JP1.9, U2.15
- net GND: now also JP3.1, JP3.2
- net N$1: now also JP1.1, U2.2; no longer JP6.1, JP6.2, JP6.3, JP6.4
- net N$2: now also JP3.5
- net N$23: now also U2.24
- net N$5: now also JP1.2, U2.3; no longer U2.26
- net N$7: now also U2.26
Other:
- board size 64 x 45.7 mm -> 111.8 x 83.8 mm
